Commit message: Added ros2_control_sim

File: description/camera.xacro (robot description, xacro)
@@ -35,5 +35,5 @@
                 <clip>
                     <near>0.05</near>
-                    <far>8.0</far>
+                    <far>15.0</far>
                 </clip>
             </camera>

File: description/lidar.xacro (robot description, xacro)
@@ -26,5 +26,5 @@
         <sensor name="laser" type="ray">
             <pose> 0 0 0 0 0 0 </pose>
-            <visualize>true</visualize>
+            <visualize>false</visualize>
             <update_rate>10</update_rate>
             <ray>
@@ -39,5 +39,5 @@
                 <range>
                     <resolution>0.01</resolution>
-                    <min>0.3</min>
+                    <min>0.5</min>
                     <max>12</max>
                 </range>

File: description/robot.urdf.xacro (robot description, xacro)
@@ -1,6 +1,12 @@
 <?xml version="1.0"?>
 <robot xmlns:xacro="http://www.ros.org/wiki/xacro"  name="robot">
+    <xacro:arg name="use_ros2_control" default="true">
     <xacro:include filename="robot_core.xacro" />
-    <xacro:include filename="gazebo_control.xacro" />
+    <xacro:if value=$(arg use_ros2_control)>
+        <xacro:include filename="ros2_control.xacro" />
+    </xacro:if>
+    <xacro:unless value=$(arg use_ros2_control)>
+        <xacro:include filename="gazebo_control.xacro" />
+    </xacro:unless>
     <xacro:include filename="lidar.xacro" />
     <xacro:include filename="camera.xacro" />

File: description/robot_core.xacro (robot description, xacro)
@@ -13,4 +13,7 @@
     <material name="black">
         <color rgba="0 0 0 1"/>
+    </material>
+    <material name="red">
+        <color rgba="1 0 0 1"/>
     </material>
     <!-- BASE LINK -->
@@ -62,5 +65,5 @@
         <collision>
             <geometry>
-                <cylinder radius="0.1" length="0.07"/>
+                <sphere radius="0.1"/>
             </geometry>
         </collision>
@@ -90,5 +93,5 @@
         <collision>
             <geometry>
-                <cylinder radius="0.1" length="0.07"/>
+                <sphere radius="0.1"/>
             </geometry>
         </collision>
@@ -118,5 +121,5 @@
         <collision>
             <geometry>
-                <cylinder radius="0.1" length="0.07"/>
+                <sphere radius="0.1"/>
             </geometry>
         </collision>
@@ -146,5 +149,5 @@
         <collision>
             <geometry>
-                <cylinder radius="0.1" length="0.07"/>
+                <sphere radius="0.1"/>
             </geometry>
         </collision>
