Commit message: Pi changes

File: description/robot.urdf.xacro (robot description, xacro)
@@ -2,4 +2,5 @@
 <robot xmlns:xacro="http://www.ros.org/wiki/xacro"  name="robot">
     <xacro:arg name="use_ros2_control" default="true">
+    <xacro:arg name="sim_mode" default="false">
     <xacro:include filename="robot_core.xacro" />
     <xacro:if value=$(arg use_ros2_control)>

File: description/ros2_control.xacro (robot description, xacro)
@@ -1,90 +1,95 @@
 <?xml version="1.0"?>
 <robot xmlns:xacro="http://www.ros.org/wiki/xacro">
-    <ros2_control name="RealRobot" type="system">
-        <hardware>
-            <plugin>gdiffdrive_arduino/DiffDriveArduino</plugin>
-            <param name="left_wheel_name">left_front_wheel_joint</param>
-            <param name="right_wheel_name">right_front_wheel_joint</param>
-            <param name="left_wheel_name">left_back_wheel_joint</param>
-            <param name="right_wheel_name">right_back_wheel_joint</param>
-            <param name="loop_rate">30</param>
-           <param name="device">/dev/ttyUSB0</param>
-            <param name="baud_rate">57600</param>
-            <param name="timeout">1000</param>
-            <param name="enc_counts_per_rev">3436</param>
-        </hardware>
-        <joint name="left_front_wheel_joint">
-            <command_interface name="velocity">
-                <param name="min">-100</param>
-                <param name="max">100</param>
-            </command_interface>
-            <state_interface name="velocity"/>
-            <state_interface name="position"/>
-        </joint>
-        <joint name="right_front_wheel_joint">
-            <command_interface name="velocity">
-                <param name="min">-100</param>
-                <param name="max">100</param>
-            </command_interface>
-            <state_interface name="velocity"/>
-            <state_interface name="position"/>
-        </joint>
-        <joint name="left_back_wheel_joint">
-            <command_interface name="velocity">
-                <param name="min">-100</param>
-                <param name="max">100</param>
-            </command_interface>
-            <state_interface name="velocity"/>
-            <state_interface name="position"/>
-        </joint>
-        <joint name="right_back_wheel_joint">
-            <command_interface name="velocity">
-                <param name="min">-100</param>
-                <param name="max">100</param>
-            </command_interface>
-            <state_interface name="velocity"/>
-            <state_interface name="position"/>
-        </joint>
-    </ros2_control>
-  <!--   <ros2_control name="GazeboSystem" type="system">
-        <hardware>
-            <plugin>gazebo_ros2_control/GazeboSystem</plugin>
-        </hardware>
-        <joint name="left_front_wheel_joint">
-            <command_interface name="velocity">
-                <param name="min">-100</param>
-                <param name="max">100</param>
-            </command_interface>
-            <state_interface name="velocity"/>
-            <state_interface name="position"/>
-        </joint>
-        <joint name="right_front_wheel_joint">
-            <command_interface name="velocity">
-                <param name="min">-100</param>
-                <param name="max">100</param>
-            </command_interface>
-            <state_interface name="velocity"/>
-            <state_interface name="position"/>
-        </joint>
-        <joint name="left_back_wheel_joint">
-            <command_interface name="velocity">
-                <param name="min">-100</param>
-                <param name="max">100</param>
-            </command_interface>
-            <state_interface name="velocity"/>
-            <state_interface name="position"/>
-        </joint>
-        <joint name="right_back_wheel_joint">
-            <command_interface name="velocity">
-                <param name="min">-100</param>
-                <param name="max">100</param>
-            </command_interface>
-            <state_interface name="velocity"/>
-            <state_interface name="position"/>
-        </joint>
-    </ros2_control> -->
+    <xacro:unless value=$(arg sim_mode)>
+        <ros2_control name="RealRobot" type="system">
+            <hardware>
+                <plugin>diffdrive_arduino/DiffDriveArduinoHardware</plugin>
+                <param name="left_wheel_name">left_front_wheel_joint</param>
+                <param name="right_wheel_name">right_front_wheel_joint</param>
+                <param name="left_wheel_name">left_back_wheel_joint</param>
+                <param name="right_wheel_name">right_back_wheel_joint</param>
+                <param name="loop_rate">30</param>
+            <param name="device">/dev/ttyUSB0</param>
+                <param name="baud_rate">57600</param>
+                <param name="timeout_ms">1000</param>
+                <param name="enc_counts_per_rev">5780</param>
+            </hardware>
+            <joint name="left_front_wheel_joint">
+                <command_interface name="velocity">
+                    <param name="min">-100</param>
+                    <param name="max">100</param>
+                </command_interface>
+                <state_interface name="velocity"/>
+                <state_interface name="position"/>
+            </joint>
+            <joint name="right_front_wheel_joint">
+                <command_interface name="velocity">
+                    <param name="min">-100</param>
+                    <param name="max">100</param>
+                </command_interface>
+                <state_interface name="velocity"/>
+                <state_interface name="position"/>
+            </joint>
+            <joint name="left_back_wheel_joint">
+                <command_interface name="velocity">
+                    <param name="min">-100</param>
+                    <param name="max">100</param>
+                </command_interface>
+                <state_interface name="velocity"/>
+                <state_interface name="position"/>
+            </joint>
+            <joint name="right_back_wheel_joint">
+                <command_interface name="velocity">
+                    <param name="min">-100</param>
+                    <param name="max">100</param>
+                </command_interface>
+                <state_interface name="velocity"/>
+                <state_interface name="position"/>
+            </joint>
+        </ros2_control>
+    </xacro:unless>
+    <xacro:if value=$(arg sim_mode)>
+        <ros2_control name="GazeboSystem" type="system">
+            <hardware>
+                <plugin>gazebo_ros2_control/GazeboSystem</plugin>
+            </hardware>
+            <joint name="left_front_wheel_joint">
+                <command_interface name="velocity">
+                    <param name="min">-100</param>
+                    <param name="max">100</param>
+                </command_interface>
+                <state_interface name="velocity"/>
+                <state_interface name="position"/>
+            </joint>
+            <joint name="right_front_wheel_joint">
+                <command_interface name="velocity">
+                    <param name="min">-100</param>
+                    <param name="max">100</param>
+                </command_interface>
+                <state_interface name="velocity"/>
+                <state_interface name="position"/>
+            </joint>
+            <joint name="left_back_wheel_joint">
+                <command_interface name="velocity">
+                    <param name="min">-100</param>
+                    <param name="max">100</param>
+                </command_interface>
+                <state_interface name="velocity"/>
+                <state_interface name="position"/>
+            </joint>
+            <joint name="right_back_wheel_joint">
+                <command_interface name="velocity">
+                    <param name="min">-100</param>
+                    <param name="max">100</param>
+                </command_interface>
+                <state_interface name="velocity"/>
+                <state_interface name="position"/>
+            </joint>
+        </ros2_control>
+    </xacro:if>
     <gazebo>
         <plugin name="gazebo_ros2_control" filename="libgazebo_ros2_control.so">
             <parameters>$(find hosbot_pkg)/config/my_controllers.yaml</parameters>
+            <parameters>$(find hosbot_pkg)/config/gaz_ros2_control_use_sim.yaml</parameters>
         </plugin>
     </gazebo>

Commit message: Hardware Interface ros2_control

File: description/robot.urdf.xacro (robot description, xacro)
@@ -1,13 +1,14 @@
 <?xml version="1.0"?>
 <robot xmlns:xacro="http://www.ros.org/wiki/xacro"  name="robot">
-    <xacro:arg name="use_ros2_control" default="true">
-    <xacro:arg name="sim_mode" default="false">
+    <xacro:arg name="use_ros2_control" default="true"/>
+    <xacro:arg name="sim_mode" default="false"/>
     <xacro:include filename="robot_core.xacro" />
-    <xacro:if value=$(arg use_ros2_control)>
+     <xacro:include filename="ros2_control.xacro" />
+<!--     <xacro:if value=$(arg use_ros2_control)>
         <xacro:include filename="ros2_control.xacro" />
     </xacro:if>
     <xacro:unless value=$(arg use_ros2_control)>
         <xacro:include filename="gazebo_control.xacro" />
-    </xacro:unless>
+    </xacro:unless> -->
     <xacro:include filename="lidar.xacro" />
     <xacro:include filename="camera.xacro" />

File: description/robot_core.xacro (robot description, xacro)
@@ -131,5 +131,5 @@
         <material>Gazebo/Blue</material>
     </gazebo>
-    <!-- RIGHT FRONT WHEEL LINK -->
+   <!-- RIGHT FRONT WHEEL LINK -->
     <joint name="right_front_wheel_joint" type="continuous">
         <parent link="base_link"/>

File: description/ros2_control.xacro (robot description, xacro)
@@ -1,5 +1,53 @@
 <?xml version="1.0"?>
 <robot xmlns:xacro="http://www.ros.org/wiki/xacro">
-    <xacro:unless value=$(arg sim_mode)>
+<ros2_control name="RealRobot" type="system">
+    <hardware>
+        <plugin>diffdrive_arduino/DiffDriveArduinoHardware</plugin>
+        <param name="left_wheel_name">left_back_wheel_joint</param>
+        <param name="right_wheel_name">right_back_wheel_joint</param>
+        <param name="loop_rate">30</param>
+        <param name="device">/dev/ttyUSB1</param>
+        <param name="baud_rate">57600</param>
+        <param name="timeout_ms">1000</param>
+        <param name="enc_counts_per_rev">5780</param>
+        <param name="pid_p">20</param>
+        <param name="pid_d">12</param>
+        <param name="pid_i">0</param>
+        <param name="pid_o">50</param>
+    </hardware>
+    <!-- <joint name="left_front_wheel_joint">
+        <command_interface name="velocity">
+            <param name="min">-100</param>
+            <param name="max">100</param>
+        </command_interface>
+        <state_interface name="velocity"/>
+        <state_interface name="position"/>
+    </joint>
+    <joint name="right_front_wheel_joint">
+        <command_interface name="velocity">
+            <param name="min">-100</param>
+            <param name="max">100</param>
+        </command_interface>
+        <state_interface name="velocity"/>
+        <state_interface name="position"/>
+    </joint> -->
+    <joint name="left_back_wheel_joint">
+        <command_interface name="velocity">
+            <param name="min">-100</param>
+            <param name="max">100</param>
+        </command_interface>
+        <state_interface name="position"/>
+        <state_interface name="velocity"/>
+    </joint>
+    <joint name="right_back_wheel_joint">
+        <command_interface name="velocity">
+            <param name="min">-100</param>
+            <param name="max">100</param>
+        </command_interface>
+        <state_interface name="position"/>
+        <state_interface name="velocity"/>
+    </joint>
+</ros2_control>
+   <!--  <xacro:unless value=$(arg sim_mode)>
         <ros2_control name="RealRobot" type="system">
             <hardware>
@@ -87,5 +135,5 @@
             </joint>
         </ros2_control>
-    </xacro:if>
+    </xacro:if> -->
     <gazebo>
         <plugin name="gazebo_ros2_control" filename="libgazebo_ros2_control.so">
