Commit message: HosBot

File: src/hosbot_pkg/description/gazebo_control.xacro (robot description, xacro)
@@ -1,29 +1,7 @@
 <?xml version="1.0"?>
 <robot xmlns:xacro="http://www.ros.org/wiki/xacro">
-    <plugin name="skid_steer_drive_controller" filename="libgazebo_ros_skid_steer_drive.so">
-        <updateRate>100.0</updateRate>
-        <robotNamespace></robotNamespace>
-        <leftFrontJoint>left_front_wheel_joint</leftFrontJoint>
-        <rightFrontJoint>right_front_wheel_joint</rightFrontJoint>
-        <leftRearJoint>left_back_wheel_joint</leftRearJoint>
-        <rightRearJoint>right_back_wheel_joint</rightRearJoint>
-        <wheelSeparation>0.65</wheelSeparation>
-        <wheelDiameter>0.2</wheelDiameter>
-        <robotBaseFrame>base_link</robotBaseFrame>
-        <torque>20</torque>
-        <topicName>cmd_vel</topicName>
-        <odometryTopic>odom</odometryTopic>
-        <odometryFrame>odom</odometryFrame>
-        <commandTopic>cmd_vel</commandTopic>
-        <topic_name_twist>cmd_vel</topic_name_twist>
-        <topic_name_odometry>odom</topic_name_odometry>
-        <topic_name_joint>joint</topic_name_joint>
-        <broadcastTF>true</broadcastTF>
-        <covariance_x>0.0001</covariance_x>
-        <covariance_y>0.0001</covariance_y>
-        <covariance_yaw>0.01</covariance_yaw>
-    </plugin>
-    <!-- <gazebo>
+    <gazebo>
         <plugin name="diff_drive" filename="libgazebo_ros_diff_drive.so">
+            <!-- Wheel Information -->
             <num_wheel_pairs>2</num_wheel_pairs>
             <left_joint>left_front_wheel_joint</left_joint>
@@ -35,10 +13,12 @@
             <wheel_diameter>0.2</wheel_diameter>
             <wheel_diameter>0.2</wheel_diameter>
+            <!-- Limits -->
             <updateRate>100</updateRate>
-            <max_wheel_torque>100</max_wheel_torque>
+            <max_wheel_torque>300</max_wheel_torque>
             <max_wheel_acceleration>1.0</max_wheel_acceleration>
-            <command_topic>cmd_vel</command_topic>
+            <!-- Output -->
+          <!--   <command_topic>cmd_vel</command_topic>
             <odometry_topic>odom</odometry_topic>
-            <odometry_frame>odom</odometry_frame>
+            <odometry_frame>odom</odometry_frame> -->
             <robot_base_frame>base_link</robot_base_frame>
             <publish_odom>true</publish_odom>
@@ -46,4 +26,4 @@
             <publish_wheel_tf>true</publish_wheel_tf>
         </plugin>
-    </gazebo> -->
+    </gazebo>
 </robot>

File: src/hosbot_pkg/description/robot_core.xacro (robot description, xacro)
@@ -21,9 +21,9 @@
         <parent link="base_link"/>
         <child link="chassis"/>
-        <origin xyz="-0.3 0 0"/>
+        <origin xyz="-0.35 0 0"/>
     </joint>
     <link name="chassis">
         <visual>
-            <origin xyz="0.3 0 0.225"/>
+            <origin xyz="0.35 0 0.225"/>
             <geometry>
                 <box size="0.7 0.6 0.45"/>
@@ -32,5 +32,5 @@
         </visual>
         <collision>
-            <origin xyz="0.15 0 0.075"/>
+            <origin xyz="0.35 0 0.225"/>
             <geometry>
                 <box size="0.7 0.6 0.45"/>
@@ -71,6 +71,4 @@
     <gazebo reference="left_back_wheel">
         <material>Gazebo/Blue</material>
-        <mu1 value="0.02"/>
-        <mu2 value="0.02"/>
     </gazebo>
     <!-- RIGHT BACK WHEEL LINK -->
@@ -101,6 +99,4 @@
     <gazebo reference="right_back_wheel">
         <material>Gazebo/Blue</material>
-        <mu1 value="0.02"/>
-        <mu2 value="0.02"/>
     </gazebo>
     <!-- LEFT FRONT WHEEL LINK -->
@@ -131,6 +127,4 @@
     <gazebo reference="left_front_wheel">
         <material>Gazebo/Blue</material>
-        <mu1 value="0.02"/>
-        <mu2 value="0.02"/>
     </gazebo>
     <!-- RIGHT FRONT WHEEL LINK -->
@@ -161,6 +155,4 @@
     <gazebo reference="right_front_wheel">
         <material>Gazebo/Blue</material>
-        <mu1 value="0.02"/>
-        <mu2 value="0.02"/>
     </gazebo>
 </robot>
